Commit message: arm integration

File: ROS_WS/src/simulation/robot/arm.xacro (robot description, xacro)
@@ -10,4 +10,11 @@
   <!-- <origin rpy="0 0 1.5707" xyz="0 0 0"/> -->
   <!-- <link name="world"/> -->
+  <link name='arm_base_link'>
+    <inertial>
+      <mass value="1e-5" />
+      <origin xyz="0 0 0" rpy="0 0 0"/>
+      <inertia ixx="1e-6" ixy="0" ixz="0" iyy="1e-6" iyz="0" izz="1e-6" />
+    </inertial>
+  </link>
   <link name='base'>
     <inertial>
@@ -34,4 +41,11 @@
     </visual>
   </link>
+  <joint type="revolute" name="base_arm_hinge">
+    <limit upper="3.14" lower="-3.14" velocity="5" effort="10000"/>
+    <origin xyz="0 0 0" rpy="0 0 0"/>
+    <axis xyz="0 0 1" />
+    <child link="base"/>
+    <parent link="arm_base_link"/>
+  </joint>
   <link name='upper_arm'>
     <collision name='collision'>
@@ -129,4 +143,11 @@
     </inertial>
   </link>
+  <gazebo reference="claw_base">
+    <implicitSpringDamper>1</implicitSpringDamper>
+    <mu1>100000</mu1>
+    <mu2>100000</mu2>
+    <kp>100000000.0</kp>
+    <kd>1.0</kd>
+  </gazebo>
   <link name='claw_right'>
     <collision name='collision'>
@@ -159,16 +180,17 @@
       </geometry>
     </visual>
-    <inertial>
+    <!-- <inertial>
       <mass value="${mass_claw}"/>
       <origin xyz="0.000025 0.019708 0.040881" rpy="0 0 0"/>
-      <!-- | 61.941238 0.000016 0.000021 |
-      | 0.000016 46.885822 -23.824060 |
-      | 0.000021 -23.824060 15.744728 |
-      | ixx ixy ixz |
-      | ixy iyy iyz |
-      | ixz iyz izz | -->
       <inertia
         ixx="${mass_claw / 0.00000743 * (61.941238*1.0e-10)}" ixy="0.0" ixz="0.0"
         iyy="${mass_claw / 0.00000743 * (46.885822*1.0e-10)}" iyz="${mass_claw / 0.0000743 * (-23.824060*1.0e-10)}" izz="${mass_claw / 0.0000743 * (15.744728*1.0e-10)}"/>
+    </inertial> -->
+    <inertial>
+        <mass value="0.018491" />
+        <origin xyz="0.0 0.0 0.0" />
+        <inertia ixx = "0.000009" ixy = "-0.000001" ixz = "0.000000"
+                  iyx = "-0.000001" iyy = "0.000001" iyz = "0.000000"
+                  izx = "0.000000" izy = "0.000000" izz = "0.000010" />
     </inertial>
   </link>
@@ -187,5 +209,5 @@
         </friction>
       </surface>
-      c<contact>
+      <contact>
         <ode>
           <mu>1.4</mu>
@@ -203,5 +225,5 @@
       </geometry>
     </visual>
-    <inertial>
+    <!-- <inertial>
       <mass value="${mass_claw}"/>
       <origin xyz="0 0.015 0.04" rpy="2.5 0 0"/>
@@ -210,8 +232,29 @@
         iyy="${mass_claw / 12.0 * (0.1*0.1 + 0.02*0.02)}" iyz="0.0"
         izz="${mass_claw / 12.0 * (0.02*0.02 + 0.02*0.02)}"/>
-    </inertial>
-  </link>
-  <joint type="continuous" name="lower_hinge">
-    <!-- <limit upper="1.57" lower="-1.57" velocity="5" effort="1000000"/> -->
+    </inertial> -->
+    <inertial>
+        <mass value="0.018491" />
+        <origin xyz="0.0 0.0 0.0" />
+        <inertia ixx = "0.000009" ixy = "-0.000001" ixz = "0.000000"
+                  iyx = "-0.000001" iyy = "0.000001" iyz = "0.000000"
+                  izx = "0.000000" izy = "0.000000" izz = "0.000010" />
+    </inertial>
+  </link>
+  <gazebo reference="claw_left">
+    <implicitSpringDamper>1</implicitSpringDamper>
+    <mu1>100000</mu1>
+    <mu2>100000</mu2>
+    <kp>100000000.0</kp>
+    <kd>1.0</kd>
+  </gazebo>
+  <gazebo reference="claw_right">
+    <implicitSpringDamper>1</implicitSpringDamper>
+    <mu1>100000</mu1>
+    <mu2>100000</mu2>
+    <kp>100000000.0</kp>
+    <kd>1.0</kd>
+  </gazebo>
+  <joint type="revolute" name="lower_hinge">
+    <limit upper="3.14" lower="-3.14" velocity="5" effort="10000"/>
     <origin xyz="0 0 0.074"/>
     <axis xyz="0 1 0" />
@@ -219,6 +262,6 @@
     <parent link="base"/>
   </joint>
-  <joint type="continuous" name="upper_hinge">
-    <!-- <limit upper="1.57" lower="-1.57" velocity="5" effort="10000"/> -->
+  <joint type="revolute" name="upper_hinge">
+    <limit upper="3.0" lower="-3.0" velocity="5" effort="10000"/>
     <origin xyz="0 0.0 0.507"/>
     <axis xyz="0 1 0" />
@@ -241,5 +284,5 @@
   </joint>
   <joint type="revolute" name="claw_right_hinge">
-    <limit upper="1.57" lower="0" velocity="0.001" effort="5"/>
+    <limit upper="1.57" lower="0" velocity="2.0" effort="1000"/>
     <origin xyz="0 -0.04175 0.128"/>
     <axis xyz="1 0 0" />
@@ -248,5 +291,5 @@
   </joint>
   <joint type="revolute" name="claw_left_hinge">
-    <limit upper="1.57" lower="0" velocity="0.1" effort="5"/>
+    <limit upper="1.57" lower="0" velocity="2.0" effort="1000"/>
     <origin xyz="0 0.04175 0.128" rpy="0 0 3.14"/>
     <axis xyz="1 0 0" />
@@ -324,3 +367,21 @@
     </actuator>
   </transmission>
+  <!--using the grasp plugin so that the gripper can grasp things in simulation-->
+  <gazebo>
+   <plugin name="gazebo_grasp_fix" filename="libgazebo_grasp_fix.so">
+        <arm>
+           <arm_name>rover_arm</arm_name>
+           <palm_link>claw_base</palm_link>
+           <gripper_link>claw_left</gripper_link>
+           <gripper_link>claw_right</gripper_link>
+        </arm>
+       <forces_angle_tolerance>100</forces_angle_tolerance>
+       <update_rate>5</update_rate>
+       <grip_count_threshold>4</grip_count_threshold>
+       <max_grip_count>8</max_grip_count>
+       <release_tolerance>0.005</release_tolerance>
+       <disable_collisions_on_attach>false</disable_collisions_on_attach>
+       <contact_topic>__default_topic__</contact_topic>
+    </plugin>
+  </gazebo>
 </robot>

File: ROS_WS/src/simulation/robot/rover2.xacro (robot description, xacro)
@@ -1,14 +1,13 @@
 <?xml version='1.0'?>
 <robot name="rover" xmlns:xacro="http://www.ros.org/wiki/xacro">
-  <xacro:include filename="$(find simulation)/robot/rover.gazebo" />
+  <xacro:include filename="$(find simulation)/robot/rover_drive.gazebo" />
   <!-- <xacro:include filename="$(find simulation)/robot/arm.xacro" /> -->
-  <origin rpy="0 0 1.5707" xyz="0 0 0"/>
+  <!-- <origin rpy="0 0 1.5707" xyz="0 0 0"/> -->
   <link name='chassis'>
     <pose>0 0 0.1 0 0 0</pose>
     <collision name='collision'>
-      <!-- <origin rpy="0 0 1.5707" xyz="-0.4 0 -0.1"/> -->
-      <origin rpy="0 0 1.5707" xyz="-0.4 0 -0.1"/>
-      <geometry>
-        <box size="0.7 1.0 0.3"/>
+      <origin rpy="0 0 0" xyz="0 0 0"/>
+      <geometry>
+        <box size="0.9 0.58 0.2"/>
       </geometry>
       <surface>
@@ -25,19 +24,148 @@
     <visual name='chassis_visual'>
       <!-- <pose>-0.25 0.18 -0.04 0 0 0</pose> -->
-      <origin rpy="0 0 0" xyz="0 0 -0.04"/>
-      <geometry>
-        <mesh filename="package://simulation/robot/chassis_with_wheels.dae"/>
+      <origin rpy="0 0 0" xyz="0 0 0"/>
+      <geometry>
+        <mesh filename="package://simulation/robot/chassis_only.dae"/>
       </geometry>
     </visual>
     <inertial>
       <mass value="20.0"/>
-      <origin xyz="0 0 -0.1" rpy=" 0 0 1.5707"/>
-      <inertia
+      <origin xyz="0.15 0 0" rpy=" 0 0 0"/>
+      <!-- <inertia
           ixx="1.0" ixy="0" ixz="0"
           iyy="1.0" iyz="0"
-          izz="0.5"
-      />
-    </inertial>
-  </link>
+          izz="1.0"
+      /> -->
+      <inertia
+          ixx="0.627" ixy="0" ixz="0"
+          iyy="1.72" iyz="0"
+          izz="1.91"/>
+    </inertial>
+  </link>
+  <link name='upper_right_suspension'>
+    <pose>0 0 0 0 0 0 </pose>
+    <collision name='collision'>
+      <origin rpy="0 0 0" xyz="0 0 0"/>
+      <geometry>
+        <mesh filename="package://simulation/robot/upper_sus.dae"/>
+      </geometry>>
+    </collision>
+    <visual name='visual'>
+      <!-- <pose>-0.25 0.18 -0.04 0 0 0</pose> -->
+      <!-- <origin rpy="0 0 0" xyz="0 0 -0.04"/> -->
+      <geometry>
+        <mesh filename="package://simulation/robot/upper_sus.dae"/>
+      </geometry>
+    </visual>
+    <inertial>
+      <mass value="1.0"/>
+      <origin xyz="0.05 0 0" rpy=" 0 0 0"/>
+      <inertia
+        ixx="1.0" ixy="0.0" ixz="0.0"
+        iyy="1.0" iyz="0.0"
+        izz="1.0"/>
+    </inertial>
+  </link>
+  <joint name="upper_right_sus_joint" type="revolute">
+    <origin xyz="0.1212 -0.3702 -0.05" rpy="0 0 3.14"/>
+    <limit upper="0.57" lower="-0.57" velocity="0.5" effort="0.5"/>
+    <axis xyz="0 1 0" />
+    <parent link="chassis"/>
+    <child link="upper_right_suspension"/>
+  </joint>
+  <link name='upper_left_suspension'>
+    <pose>0 0 0 0 0 0</pose>
+    <collision name='collision'>
+      <origin rpy="0 0 0" xyz="0 0 0"/>
+      <geometry>
+        <mesh filename="package://simulation/robot/upper_sus.dae"/>
+      </geometry>>
+    </collision>
+    <visual name='visual'>
+      <!-- <pose>-0.25 0.18 -0.04 0 0 0</pose> -->
+      <!-- <origin rpy="0 0 0" xyz="0 0 -0.04"/> -->
+      <geometry>
+        <mesh filename="package://simulation/robot/upper_sus.dae"/>
+      </geometry>
+    </visual>
+    <inertial>
+      <mass value="1.0"/>
+      <origin xyz="0 0 0" rpy=" 0 0 0"/>
+      <inertia
+        ixx="1.0" ixy="0.0" ixz="0.0"
+        iyy="1.0" iyz="0.0"
+        izz="1.0"/>
+    </inertial>
+  </link>
+  <joint name="upper_left_sus_joint" type="revolute">
+    <origin xyz="0.1212 0.3102 -0.05" rpy="0 0 3.14"/>
+    <limit upper="0.57" lower="-0.57" velocity="0.5" effort="0.5"/>
+    <axis xyz="0 1 0" />
+    <parent link="chassis"/>
+    <child link="upper_left_suspension"/>
+  </joint>
+  <link name='lower_right_suspension'>
+    <pose>0 0 0 0 0 0</pose>
+    <collision name='collision'>
+      <origin rpy="0 0 0" xyz="0 0 0"/>
+      <geometry>
+        <mesh filename="package://simulation/robot/lower_sus.dae"/>
+      </geometry>>
+    </collision>
+    <visual name='visual'>
+      <!-- <pose>-0.25 0.18 -0.04 0 0 0</pose> -->
+      <!-- <origin rpy="0 0 0" xyz="0 0 -0.04"/> -->
+      <geometry>
+        <mesh filename="package://simulation/robot/lower_sus.dae"/>
+      </geometry>
+    </visual>
+    <inertial>
+      <mass value="1.0"/>
+      <origin xyz="0 0 0" rpy=" 0 0 0"/>
+      <inertia
+        ixx="1.0" ixy="0.0" ixz="0.0"
+        iyy="1.0" iyz="0.0"
+        izz="1.0"/>
+    </inertial>
+  </link>
+  <joint name="lower_right_sus_joint" type="revolute">
+    <origin xyz="-0.3864 -0.01 -0.1035" rpy="0 0 0"/>
+    <axis xyz="0 1 0" />
+    <limit upper="0.57" lower="-0.57" velocity="0.5" effort="0.5"/>
+    <dynamics friction="0.9"/>
+    <parent link="upper_right_suspension"/>
+    <child link="lower_right_suspension"/>
+  </joint>
+  <link name='lower_left_suspension'>
+    <pose>0 0 0 0 0 0</pose>
+    <collision name='collision'>
+      <origin rpy="0 0 0" xyz="0 0 0"/>
+      <geometry>
+        <mesh filename="package://simulation/robot/lower_sus.dae"/>
+      </geometry>>
+    </collision>
+    <visual name='visual'>
+      <!-- <pose>-0.25 0.18 -0.04 0 0 0</pose> -->
+      <!-- <origin rpy="0 0 0" xyz="0 0 -0.04"/> -->
+      <geometry>
+        <mesh filename="package://simulation/robot/lower_sus.dae"/>
+      </geometry>
+    </visual>
+    <inertial>
+      <mass value="1.0"/>
+      <origin xyz="0 0 0" rpy=" 0 0 0"/>
+      <inertia
+        ixx="1.0" ixy="0.0" ixz="0.0"
+        iyy="1.0" iyz="0.0"
+        izz="1.0"/>
+    </inertial>
+  </link>
+  <joint name="lower_left_sus_joint" type="revolute">
+    <origin xyz="-0.3864 -0.01 -0.1035" rpy="0 0 0"/>
+    <limit upper="0.57" lower="-0.57" velocity="0.5" effort="0.5"/>
+    <axis xyz="0 1 0" />
+    <parent link="upper_left_suspension"/>
+    <child link="lower_left_suspension"/>
+  </joint>
   <!-- <link name='base_footprint'></link>
   <joint name="base_footprint_joint" type="fixed">
@@ -53,6 +181,5 @@
   </joint> -->
   <!-- Kinect Link -->
-  <link name='kinect_link'>
-    <!-- <pose>0 0.25 0 0 0 0</pose> -->
+  <!-- <link name='kinect_link'>
     <inertial>
       <origin xyz="0 0 0" rpy="0 0 0"/>
@@ -78,7 +205,7 @@
     <parent link="chassis"/>
     <child link="kinect_link"/>
-  </joint>
+  </joint> -->
   <!-- Camera -->
-  <link name="camera_link1">
+  <!-- <link name="camera_link1">
     <collision>
       <origin xyz="0 0 0" rpy="0 0 0"/>
@@ -105,7 +232,7 @@
     <parent link="chassis"/>
     <child link="camera_link1"/>
-  </joint>
+  </joint> -->
     <!-- Camera -->
-  <link name="camera_link2">
+  <!-- <link name="camera_link2">
     <collision>
       <origin xyz="0 0 0" rpy="0 0 0"/>
@@ -132,5 +259,5 @@
     <parent link="chassis"/>
     <child link="camera_link2"/>
-  </joint>
+  </joint> -->
   <!-- Hokuyo Laser -->
   <!-- <link name="hokuyo_link">
@@ -184,5 +311,5 @@
   </joint> -->
   <!-- GPS sensor -->
-  <link name="gps_link">
+  <!-- <link name="gps_link">
     <inertial>
       <mass value="1e-5" />
@@ -206,6 +333,6 @@
     <parent link="chassis"/>
     <child link="gps_link"/>
-  </joint>
-  <link name="left_wheel">
+  </joint> -->
+  <link name="middle_left_wheel">
     <!-- <origin xyz="0.5 0.145 -0.31" rpy="0 1.5707 0"/> -->
     <collision name="collision">
@@ -255,5 +382,5 @@
     </inertial>
   </link>
-  <link name="right_wheel">
+  <link name="middle_right_wheel">
     <!-- <origin xyz="-0.44 0.145 -0.31" rpy="0 1.5707 0"/> -->
     <collision name="collision">
@@ -279,4 +406,50 @@
     </inertial>
   </link>
+  <link name="back_left_wheel">
+    <collision name="collision">
+      <origin xyz="0 0 0" rpy="0 0 0"/>
+      <geometry>
+        <cylinder radius="0.1" length="0.05"/>
+      </geometry>
+    </collision>
+    <visual name="visual">
+      <origin xyz="0 0 0" rpy="0 0 0"/>
+      <geometry>
+        <cylinder radius="0.1" length="0.05"/>
+      </geometry>
+    </visual>
+    <inertial>
+      <origin xyz="0 0 0" rpy="0 0 0"/>
+      <mass value="5"/>
+      <cylinder_inertia m="5" r="0.1" h="0.05"/>
+      <inertia
+        ixx="1.0" ixy="0.0" ixz="0.0"
+        iyy="1.0" iyz="0.0"
+        izz="1.0"/>
+    </inertial>
+  </link>
+  <link name="back_right_wheel">
+    <collision name="collision">
+      <origin xyz="0 0 0" rpy="0 0 0"/>
+      <geometry>
+        <cylinder radius="0.1" length="0.05"/>
+      </geometry>
+    </collision>
+    <visual name="visual">
+      <origin xyz="0 0 0" rpy="0 0 0"/>
+      <geometry>
+        <cylinder radius="0.1" length="0.05"/>
+      </geometry>
+    </visual>
+    <inertial>
+      <origin xyz="0 0 0" rpy="0 0 0"/>
+      <mass value="5"/>
+      <cylinder_inertia m="5" r="0.1" h="0.05"/>
+      <inertia
+        ixx="1.0" ixy="0.0" ixz="0.0"
+        iyy="1.0" iyz="0.0"
+        izz="1.0"/>
+    </inertial>
+  </link>
   <link name="front_right_wheel">
     <!-- <origin xyz="-0.44 -0.468 -0.38" rpy="0 1.5707 0"/> -->
@@ -303,35 +476,51 @@
     </inertial>
   </link>
-  <joint type="continuous" name="left_wheel_hinge">
-    <origin xyz="0.045 0.49 -0.41" rpy="0 1.5707 1.5707"/>
-    <child link="left_wheel"/>
-    <parent link="chassis"/>
+  <joint type="continuous" name="middle_left_wheel_hinge">
+    <origin xyz="0.3 -0.09 -0.1593" rpy="0 -1.5707 1.5707"/>
+    <child link="middle_left_wheel"/>
+    <parent link="lower_left_suspension"/>
     <axis xyz="0 0 1" rpy="0 0 0"/>
     <limit effort="100" velocity="100"/>
     <joint_properties damping="0.0" friction="0.0"/>
   </joint>
-  <joint type="continuous" name="front_left_wheel_hinge">
-    <origin xyz="0.64 0.49 -0.38" rpy="0 1.5707 1.5707"/>
+  <joint type="continuous" name="back_left_wheel_hinge">
+    <origin xyz="-0.3 -0.09 -0.1593" rpy="0 -1.5707 1.5707"/>
     <child link="front_left_wheel"/>
-    <parent link="chassis"/>
+    <parent link="lower_left_suspension"/>
     <axis xyz="0 0 1" rpy="0 0 0"/>
     <limit effort="100" velocity="100"/>
     <joint_properties damping="0.0" friction="0.0"/>
   </joint>
-  <joint type="continuous" name="front_right_wheel_hinge">
-    <origin xyz="0.64 -0.48 -0.38" rpy="0 1.5707 1.5707"/>
-    <child link="front_right_wheel"/>
-    <parent link="chassis"/>
+  <joint type="continuous" name="front_left_wheel_hinge">
+    <origin xyz="0.5136 -0.101 -0.237" rpy="0 -1.5707 1.5707"/>
+    <child link="back_left_wheel"/>
+    <parent link="upper_left_suspension"/>
     <axis xyz="0 0 1" rpy="0 0 0"/>
     <limit effort="100" velocity="100"/>
     <joint_properties damping="0.0" friction="0.0"/>
   </joint>
-  <joint type="continuous" name="right_wheel_hinge">
-    <origin xyz="0.045 -0.48 -0.41" rpy="0 1.5707 1.5707"/>
-    <child link="right_wheel"/>
-    <parent link="chassis"/>
+  <joint type="continuous" name="front_right_wheel_hinge">
+    <origin xyz="0.5136 0.051 -0.237" rpy="0 -1.5707 1.5707"/>
+    <child link="back_right_wheel"/>
+    <parent link="upper_right_suspension"/>
     <axis xyz="0 0 1" rpy="0 0 0"/>
     <limit effort="100" velocity="100"/>
     <joint_properties damping="0.0" friction="0.0"/>
   </joint>
+  <joint type="continuous" name="middle_right_wheel_hinge">
+    <origin xyz="0.3 0.05 -0.1593" rpy="0 -1.5707 1.5707"/>
+    <child link="middle_right_wheel"/>
+    <parent link="lower_right_suspension"/>
+    <axis xyz="0 0 1" rpy="0 0 0"/>
+    <limit effort="100" velocity="100"/>
+    <joint_properties damping="0.0" friction="0.0"/>
+  </joint>
+  <joint type="continuous" name="back_right_wheel_hinge">
+    <origin xyz="-0.3 0.05 -0.1593" rpy="0 -1.5707 1.5707"/>
+    <child link="front_right_wheel"/>
+    <parent link="lower_right_suspension"/>
+    <axis xyz="0 0 1" rpy="0 0 0"/>
+    <limit effort="100" velocity="100"/>
+    <joint_properties damping="0.0" friction="0.0"/>
+  </joint>
 </robot>

File: ROS_WS/src/simulation/robot/rover_model.xacro (robot description, xacro)
@@ -30,4 +30,10 @@
     </visual>
   </link>
+  <link name='base_footprint'><link/>
+  <joint name="base_footprint_joint" type="fixed">
+    <origin xyz="0 0 0.51" rpy="0 0 0"/>
+    <parent link="base_footprint"/>
+    <child link="chassis"/>
+  </joint>
   <link name='kinect_link'>
     <!-- <pose>0 0.25 0 0 0 0</pose> -->

File: ROS_WS/src/simulation/robot/rover_with_arm.xacro (robot description, xacro)
@@ -7,5 +7,5 @@
     <pose>0 0 0.1 0 0 0</pose>
     <collision name='collision'>
-      <origin rpy="0 0 1.5707" xyz="-0.4 0 -0.1"/>
+      <origin rpy="0 0 1.5707" xyz="0 0 -0.1"/>
       <geometry>
         <box size="0.7 1.0 0.3"/>
@@ -40,8 +40,7 @@
   </link>
   <!-- Arm joint -->
-  <joint type="continuous" name="base_arm_hinge">
+  <joint type="fixed" name="arm_joint">
     <origin xyz="0.3372 0 0.0637" rpy="0 0 0"/>
-    <axis xyz="0 0 1" />
-    <child link="base"/>
+    <child link="arm_base_link"/>
     <parent link="chassis"/>
   </joint>
@@ -88,9 +87,9 @@
       <material name="red"/>
     </visual>
-    <inertial>
-      <mass value="1e-5" />
-      <origin xyz="0 0 0" rpy="0 0 0"/>
-      <inertia ixx="1e-6" ixy="0" ixz="0" iyy="1e-6" iyz="0" izz="1e-6" />
-    </inertial>
+      <inertial>
+        <mass value="1e-5" />
+        <origin xyz="0 0 0" rpy="0 0 0"/>
+        <inertia ixx="1e-6" ixy="0" ixz="0" iyy="1e-6" iyz="0" izz="1e-6" />
+      </inertial>
   </link>
   <joint name="camera_joint1" type="fixed">
