Commit message: adjusted URDF based on real world measurments

File: ROS_WS/src/bringup/urdf/mech/base.urdf.xacro (robot description, xacro)
@@ -5,5 +5,5 @@
     <link name="base_link">
       <visual>
-        <origin xyz="0 0 ${height/2}" rpy="0 0 0"/>
+        <origin xyz="0 0 ${-height/2}" rpy="0 0 0"/>
         <geometry>
           <box size="${length} ${width} ${height}"/>

File: ROS_WS/src/bringup/urdf/rover.urdf.xacro (robot description, xacro)
@@ -8,5 +8,5 @@
   <xacro:include filename="$(find bringup)/urdf/rover_properties.urdf.xacro" />
   <xacro:base length="${base_length}" width="${base_width}" height="${base_height}" base_height= "${base_top}" />
-  <xacro:imu x_pos="${imu_pos_x}" y_pos="${imu_pos_y}" z_pos="${imu_pos_z}" />
+  <xacro:imu x_pos="${imu_pos_x}" y_pos="${imu_pos_y}" z_pos="${imu_pos_z}" yaw_pos="${imu_pos_yaw}"/>
   <xacro:d435 x_pos="${d435_pos_x}" y_pos="${d435_pos_y}" z_pos="${d435_pos_z}" />
   <xacro:gps x_pos="${gps_pos_x}" y_pos="${gps_pos_y}" z_pos="${gps_pos_z}" />

File: ROS_WS/src/bringup/urdf/rover_properties.urdf.xacro (robot description, xacro)
@@ -4,11 +4,12 @@
   <xacro:property name="base_width" value="0.8" />
   <xacro:property name="base_height" value="0.4" />
-  <xacro:property name="base_top" value="0.045" />
-  <xacro:property name="imu_pos_x" value="-0.115" />
-  <xacro:property name="imu_pos_y" value="0.05" />
-  <xacro:property name="imu_pos_z" value="0.0" />
-  <xacro:property name="d435_pos_x" value="-0.2" />
+  <xacro:property name="base_top" value="0.565" />
+  <xacro:property name="imu_pos_x" value="-0.03" />
+  <xacro:property name="imu_pos_y" value="0.245" />
+  <xacro:property name="imu_pos_z" value="-0.12" />
+  <xacro:property name="imu_pos_yaw" value="3.14" />
+  <xacro:property name="d435_pos_x" value="-0.27" />
   <xacro:property name="d435_pos_y" value="0.0" />
-  <xacro:property name="d435_pos_z" value="0.6" />
+  <xacro:property name="d435_pos_z" value="0.35" />
   <xacro:property name="gps_pos_x" value="-0.15" />
   <xacro:property name="gps_pos_y" value="0.0" />

File: ROS_WS/src/bringup/urdf/sensors/imu.urdf.xacro (robot description, xacro)
@@ -1,9 +1,9 @@
 <robot xmlns:xacro="http://ros.org/wiki/xacro">
-  <xacro:macro name="imu" params="x_pos y_pos z_pos">
+  <xacro:macro name="imu" params="x_pos y_pos z_pos yaw_pos">
     <link name="imu_link"/>
     <joint name="imu_to_base_link" type="fixed">
       <parent link="base_link"/>
       <child link="imu_link"/>
-      <origin xyz="${x_pos} ${y_pos} ${z_pos}" rpy="0 0 0"/>
+      <origin xyz="${x_pos} ${y_pos} ${z_pos}" rpy="0 0 ${yaw_pos}"/>
     </joint>
   </xacro:macro>
