Commit message: updated gps transform

File: ROS_WS/src/bringup/urdf/rover_properties.urdf.xacro (robot description, xacro)
@@ -12,6 +12,6 @@
   <xacro:property name="d435_pos_y" value="0.0" />
   <xacro:property name="d435_pos_z" value="0.35" />
-  <xacro:property name="gps_pos_x" value="-0.15" />
-  <xacro:property name="gps_pos_y" value="0.0" />
-  <xacro:property name="gps_pos_z" value="0.3" />
+  <xacro:property name="gps_pos_x" value="-0.28" />
+  <xacro:property name="gps_pos_y" value="0.26" />
+  <xacro:property name="gps_pos_z" value="0.5" />
 </robot>
